Commit message: refined urdf model, adding  a frame to specify desired end effector pose

File: URDF_model/Custom_homemade_robot.urdf (robot description, URDF)
Before this commit: robot robot, 7 links, 6 joints
Links:
- added link ee, mass 1e-9
Joints:
- added joint ee_frame: type fixed, parent link5, child ee, origin xyz=0.0100555 -0.176742 -0.0318922 rpy=-1.5708 0 1.5708, axis 0 0 0
- joint joint4: limit lower=-1.55334 upper=1.58825 effort=10 velocity=10 -> lower=-1.5708 upper=1.5708 effort=10 velocity=10
- joint joint5: limit lower=-1.55334 upper=1.58825 effort=10 velocity=10 -> lower=-1.5708 upper=1.5708 effort=10 velocity=10
